File: hardware/jd2oscope/5VRegulator.kicad_sch (KiCad schematic)
At the start: 11 parts, among them J1 9V_CONN, U3 NCP1117-5.0_SOT223

Commit message: feat: lot of progress
added decoupling caps, implemented a lot more of the comm. protocol stuffs, updated BNC connector to updated version, added more notes for GPIO pin I/O for future code implementation, lot of other stuff too (frankly can't remember all of it lol); I commit here b/c want to back up progress b/4 I go get smth to eat ;)
Parts:
- removed C4, C5: 0.1u, Capacitor_SMD:C_0603_1608Metric_Pad1.08x0.95mm_HandSolder, symbol Device:C
- removed J1: 9V_CONN, symbol lockBuster:Conn_PP3
- removed S3: JS202011SCQN, digikey-footprints:Switch_Slide_JS202011SCQN, symbol dk_Slide-Switches:JS202011SCQN
- added J4: 9V_CONN, symbol lockBuster:Conn_PP3
Connections:
- net GND: now also J4.1 (Pin_1)
- net at D1.1: now also BT1., J4.2 (Pin_2)
- no-connect marks 4 -> 0
Other:
- note removed: "Capacitor Information: 0.1u = Ceramic 10u = Electrolytic"
- moved on the sheet: C2, C3
