File: hardware/jd2oscope/jd2oscope.kicad_sch (KiCad schematic)
At the start: 4 parts, among them U1 ESP32-DEVKITC-32D

Commit message: fix: added NCs
forgot to add NCs to Wroom32 dev board; they are now added!
Connections:
- no-connect marks 0 -> 11
Changed lines of the file:
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@@
 		(color 0 0 0 0)
+	)
+	(no_connect
+		(at 134.62 67.31)
+	)
+	(no_connect
+		(at 93.98 74.93)
+	)
+	(no_connect
+		(at 134.62 77.47)
+	)
+	(no_connect
+		(at 134.62 74.93)
+	)
+	(no_connect
+		(at 134.62 72.39)
+	)
+	(no_connect
+		(at 93.98 34.29)
+	)
+	(no_connect
+		(at 134.62 41.91)
+	)
+	(no_connect
+		(at 134.62 39.37)
+	)
+	(no_connect
+		(at 134.62 64.77)
+	)
+	(no_connect
+		(at 93.98 69.85)
+	)
+	(no_connect
+		(at 93.98 72.39)
 	)
 	(wire
