File: hardware/jd2oscope/reg5V.kicad_sch (KiCad schematic)
At the start: 10 parts, among them J1 9V_CONN, U3 NCP1117-5.0_SOT223

Commit message: fix: undid the thing that I thought was a fix
it is actually 12b still lol
Other:
- title: 2CH 1MS/s 14b 50kHz 5V Oscope w/320x240 TFT & ESP32 -> 2CH 1MS/s 12b 50kHz 5V Oscope w/320x240 TFT & ESP32
Changed lines of the file:
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@@
 	(paper "A4")
 	(title_block
-		(title "2CH 1MS/s 14b 50kHz 5V Oscope w/320x240 TFT & ESP32")
+		(title "2CH 1MS/s 12b 50kHz 5V Oscope w/320x240 TFT & ESP32")
 		(date "2025-02-26")
 		(rev "1")

Commit message: fix: schematic labels
Other:
- title: 2CH 1MS/s 12b 50kHz 5V Oscope w/320x240 TFT & ESP32 -> 2CH 1MS/s 14b 50kHz 5V Oscope w/320x240 TFT & ESP32
Changed lines of the file:
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@@
 	(paper "A4")
 	(title_block
-		(title "2CH 1MS/s 12b 50kHz 5V Oscope w/320x240 TFT & ESP32")
+		(title "2CH 1MS/s 14b 50kHz 5V Oscope w/320x240 TFT & ESP32")
 		(date "2025-02-26")
 		(rev "1")
