File: hardware/jd2oscope/reg5V.kicad_sch (KiCad schematic)
At the start: 10 parts, among them J1 9V_CONN, U3 NCP1117-5.0_SOT223

Commit message: feat: filled in title block
added relevant information to schematic title block blurb in the lower right
Other:
- title: (none) -> 2CH 1MS/s 12b 50kHz 5V Oscope w/320x240 TFT & ESP32
Changed lines of the file:
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@@
 	(generator_version "8.0")
 	(paper "A4")
+	(title_block
+		(title "2CH 1MS/s 12b 50kHz 5V Oscope w/320x240 TFT & ESP32")
+		(date "2025-02-26")
+		(rev "1")
+	)
 	(junction
 		(at 167.64 85.09)

Commit message: fix: propagated group name to all sheets
before it was just on the root; forgot to click the "apply to all sheets" textbox thingie
Other:
- company: (none) -> Group 15
Changed lines of the file:
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@@
 		(date "2025-02-26")
 		(rev "1")
+		(company "Group 15")
 	)
 	(junction

Commit message: feat: updated capacitor values
and other fixes too
Parts:
- C4, C6: value 0.1u -> 100nF
- C5, C7: value 10u -> 10uF
- R2: value 560 -> 560R
Other:
- note added: "Decoupling Capacitor Information: 100nF = Ceramic 10uF = Electrolytic"
- note removed: "Decoupling Capacitor Information: 0.1u = Ceramic 10u = Electrolytic"
Changed lines of the file:
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@@
 		)
 	)
-	(text "Decoupling Capacitor Information:\n0.1u = Ceramic\n10u = Electrolytic"
+	(text "Decoupling Capacitor Information:\n100nF = Ceramic\n10uF = Electrolytic"
 		(exclude_from_sim no)
 		(at 76.962 65.532 0)
@@
 			)
 		)
-		(property "Value" "0.1u"
+		(property "Value" "100nF"
 			(at 163.83 102.8699 0)
 			(effects
@@
 			)
 		)
-		(property "Value" "10u"
+		(property "Value" "10uF"
 			(at 177.8 102.8699 0)
 			(effects
@@
 			)
 		)
-		(property "Value" "0.1u"
+		(property "Value" "100nF"
 			(at 133.35 102.8699 0)
 			(effects
@@
 			)
 		)
-		(property "Value" "560"
+		(property "Value" "560R"
 			(at 115.57 97.7899 0)
 			(effects
@@
 			)
 		)
-		(property "Value" "10u"
+		(property "Value" "10uF"
 			(at 147.32 102.8699 0)
 			(effects
