File: hardware/jd2oscope/buttonModule.kicad_sch (KiCad schematic)
At the start: 1 part

Commit message: feat: filled in title block
added relevant information to schematic title block blurb in the lower right
Other:
- title: (none) -> 2CH 1MS/s 12b 50kHz 5V Oscope w/320x240 TFT & ESP32
Changed lines of the file:
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@@
 	(generator_version "8.0")
 	(paper "A4")
+	(title_block
+		(title "2CH 1MS/s 12b 50kHz 5V Oscope w/320x240 TFT & ESP32")
+		(date "2025-02-26")
+		(rev "1")
+	)
 	(no_connect
 		(at 144.78 101.6)

Commit message: fix: propagated group name to all sheets
before it was just on the root; forgot to click the "apply to all sheets" textbox thingie
Other:
- company: (none) -> Group 15
Changed lines of the file:
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@@
 		(date "2025-02-26")
 		(rev "1")
+		(company "Group 15")
 	)
 	(no_connect

Commit message: fix: schematic labels
Other:
- title: 2CH 1MS/s 12b 50kHz 5V Oscope w/320x240 TFT & ESP32 -> 2CH 1MS/s 14b 50kHz 5V Oscope w/320x240 TFT & ESP32
Changed lines of the file:
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@@
 	(paper "A4")
 	(title_block
-		(title "2CH 1MS/s 12b 50kHz 5V Oscope w/320x240 TFT & ESP32")
+		(title "2CH 1MS/s 14b 50kHz 5V Oscope w/320x240 TFT & ESP32")
 		(date "2025-02-26")
 		(rev "1")

Commit message: fix: undid the thing that I thought was a fix
it is actually 12b still lol
Other:
- title: 2CH 1MS/s 14b 50kHz 5V Oscope w/320x240 TFT & ESP32 -> 2CH 1MS/s 12b 50kHz 5V Oscope w/320x240 TFT & ESP32
Changed lines of the file:
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@@
 	(paper "A4")
 	(title_block
-		(title "2CH 1MS/s 14b 50kHz 5V Oscope w/320x240 TFT & ESP32")
+		(title "2CH 1MS/s 12b 50kHz 5V Oscope w/320x240 TFT & ESP32")
 		(date "2025-02-26")
 		(rev "1")
